File: Keithley_177_power_repair.sch (KiCad schematic (older format))
At the start: 8 parts, among them T1 RAC20-DK, T101 Transfomer, U1 R-78E5.0-1.0

Commit message: spell check transformer
Parts:
- T101: value Transfomer -> Transformer
Other:
- note added: "Transformer Replacement"
- note removed: "Transfomer Replacement"
Changed lines of the file:
@@
 EESchema Schematic File Version 4
+LIBS:Keithley_177_power_repair-cache
 EELAYER 26 0
 EELAYER END
@@
 P 4300 2900
 F 0 "T101" H 4500 2600 60  0000 C CNN
-F 1 "Transfomer" H 4300 3200 60  0001 C CNN
+F 1 "Transformer" H 4300 3200 60  0001 C CNN
 F 2 "" H 4600 2950 60  0001 C CNN
 F 3 "" H 4600 2950 60  0001 C CNN
@@
 P 6450 2750
 F 0 "T101" H 6550 2450 60  0000 L CNN
-F 1 "Transfomer" H 6200 3050 60  0001 L CNN
+F 1 "Transformer" H 6200 3050 60  0001 L CNN
 F 2 "" H 6750 2800 60  0001 C CNN
 F 3 "" H 6750 2800 60  0001 C CNN
@@
 Connection ~ 5850 2950
 Text Notes 4000 2200 0    50   ~ 0
-Transfomer Replacement
+Transformer Replacement
 Wire Notes Line
 	4000 2200 6900 2200

Commit message: assign footprints
Parts:
- CR103: footprint (none) -> Keithley_Components:Bridge_Rectifier_Inline
- CR104: footprint (none) -> Keithley_Components:Bridge_Rectifier_Square
- T1: footprint (none) -> Keithley_Components:RAC20-K
- T101: footprint (none) -> Keithley_Components:Keithley_Transformer
- VR101, VR102, VR103: footprint (none) -> Keithley_Components:Voltage_Regulator
Connections:
- net N: now reaches T1.1 (N), T101.8 (Neutral)
- net L: now reaches T1.2 (L), T101.11 (Line)
Changed lines of the file:
@@
 F 0 "T1" H 5600 2650 50  0000 C CNN
 F 1 "RAC20-DK" H 5350 3050 50  0000 C CNN
-F 2 "" H 5250 2850 50  0001 C CNN
+F 2 "Keithley_Components:RAC20-K" H 5250 2850 50  0001 C CNN
 F 3 "" H 5250 2850 50  0001 C CNN
 	1    5350 2850
@@
 F 0 "CR103" H 4450 4100 50  0000 C CNN
 F 1 "JUMPERS" H 4791 4055 50  0001 L CNN
-F 2 "" H 4450 4100 50  0001 C CNN
+F 2 "Keithley_Components:Bridge_Rectifier_Inline" H 4450 4100 50  0001 C CNN
 F 3 "~" H 4450 4100 50  0001 C CNN
 	1    4450 4100
@@
 F 0 "CR104" H 4450 5150 50  0000 C CNN
 F 1 "JUMPERS" H 4791 5105 50  0001 L CNN
-F 2 "" H 4450 5150 50  0001 C CNN
+F 2 "Keithley_Components:Bridge_Rectifier_Square" H 4450 5150 50  0001 C CNN
 F 3 "~" H 4450 5150 50  0001 C CNN
 	1    4450 5150
@@
 F 0 "T101" H 4500 2600 60  0000 C CNN
 F 1 "Transformer" H 4300 3200 60  0001 C CNN
-F 2 "" H 4600 2950 60  0001 C CNN
+F 2 "Keithley_Components:Keithley_Transformer" H 4600 2950 60  0001 C CNN
 F 3 "" H 4600 2950 60  0001 C CNN
 	1    4300 2900
@@
 F 0 "T101" H 6550 2450 60  0000 L CNN
 F 1 "Transformer" H 6200 3050 60  0001 L CNN
-F 2 "" H 6750 2800 60  0001 C CNN
+F 2 "Keithley_Components:Keithley_Transformer" H 6750 2800 60  0001 C CNN
 F 3 "" H 6750 2800 60  0001 C CNN
 	2    6450 2750
@@
 F 0 "VR101" H 6250 4025 50  0000 C CNN
 F 1 "L7805" H 6400 4025 50  0000 L CNN
-F 2 "" H 6425 3750 50  0001 L CIN
+F 2 "Keithley_Components:Voltage_Regulator" H 6425 3750 50  0001 L CIN
 F 3 "http://www.st.com/content/ccc/resource/technical/document/datasheet/41/4f/b3/b0/12/d4/47/88/CD00000444.pdf/files/CD00000444.pdf/jcr:content/translations/en.CD00000444.pdf" H 6400 3850 50  0001 C CNN
 	1    6400 3900
@@
 F 0 "VR102" H 5250 4075 50  0000 C CNN
 F 1 "L7815" H 5400 4075 50  0000 L CNN
-F 2 "" H 5425 3800 50  0001 L CIN
+F 2 "Keithley_Components:Voltage_Regulator" H 5425 3800 50  0001 L CIN
 F 3 "http://www.st.com/content/ccc/resource/technical/document/datasheet/41/4f/b3/b0/12/d4/47/88/CD00000444.pdf/files/CD00000444.pdf/jcr:content/translations/en.CD00000444.pdf" H 5400 3900 50  0001 C CNN
 	1    5400 3950
@@
 F 0 "VR103" H 5250 4875 50  0000 C CNN
 F 1 "L7915" H 5400 4875 50  0000 L CNN
-F 2 "" H 5400 4800 50  0001 C CIN
+F 2 "Keithley_Components:Voltage_Regulator" H 5400 4800 50  0001 C CIN
 F 3 "http://www.st.com/content/ccc/resource/technical/document/datasheet/c9/16/86/41/c7/2b/45/f2/CD00000450.pdf/files/CD00000450.pdf/jcr:content/translations/en.CD00000450.pdf" H 5400 5000 50  0001 C CNN
 	1    5400 5000
@@
 Wire Notes Line
 	7050 3550 7050 5250
+Text Label 4700 2750 0    50   ~ 0
+L
+Text Label 4700 3050 0    50   ~ 0
+N
 $EndSCHEMATC

Commit message: remove links
Parts:
- removed CR103: JUMPERS, Keithley_Components:Bridge_Rectifier_Inline, symbol Device:D_Bridge_+AA-
- removed CR104: JUMPERS, Keithley_Components:Bridge_Rectifier_Square, symbol Device:D_Bridge_+AA-
- removed VR102: L7815, Keithley_Components:Voltage_Regulator, symbol Regulator_Linear:L7815
- removed VR103: L7915, Keithley_Components:Voltage_Regulator, symbol Regulator_Linear:L7915
- added TP1: +15V, TestPoint:TestPoint_Pad_D2.0mm, symbol Connector:TestPoint
- added TP2: -15V, TestPoint:TestPoint_Pad_D2.0mm, symbol Connector:TestPoint
- added TP3: 5V, TestPoint:TestPoint_Pad_D2.0mm, symbol Connector:TestPoint
Connections:
- net +15V: now also TP1.1
- net -15V: now also TP2.1
- net GND: now reaches T1.4 (Com), T101.3 (Gnd_7805), T101.5 (GND)
- net at U1.3 (OUT), VR101.3 (OUT): now also TP3.1
- no-connect marks 2 -> 0
Other:
- note removed: "CR103 Jumpers"
- note removed: "CR104 Jumpers"
- note removed: "VR102 Jumpers"
- note removed: "VR103 Jumpers"
- moved on the sheet: U1, VR101
